Commit message: updated

File: assignment_2/drive_bot/urdf/trail_robo.urdf (robot description, URDF)
Before this commit: robot trail_robo, 5 links, 4 joints
Links:
- link chassis: geometry collision box size=0.4 0.4 0.1; collision sphere radius=0.05
Joints:
- joint camera_head_joint: origin xyz=0.225 0 0.0725 rpy=0.0 0 0 -> xyz=0.175 0 0.0725 rpy=0.0 0 0
- joint joint_left_wheel: origin xyz=-0.2 0.201 0 rpy=0 0 0 -> xyz=0 0.201 0 rpy=0 0 0
- joint joint_right_wheel: origin xyz=-0.2 -0.201 0 rpy=0 0 0 -> xyz=0 -0.201 0 rpy=0 0 0

Commit message: final code

File: assignment_2/drive_bot/urdf/trail_robo.urdf (robot description, URDF)
Before this commit: robot trail_robo, 5 links, 4 joints
Links:
- link chassis: geometry collision box size=0.4 0.4 0.1; collision sphere radius=0.049
